File: nenad_struja.kicad_sch (KiCad schematic)
At the start: 29 parts, among them Q1 MMBT5551L, Q2 MMBT5551L

Commit message: dodao pcb dizajn
Parts:
- C1, C2, C3, C4, C5, C6, C7, C8: footprint Capacitor_SMD:C_0603_1608Metric -> (none)
- R1, R10, R11, R12, R13, R2, R3, R4, R5, R6, R7, R8, R9: footprint Resistor_SMD:R_0603_1608Metric -> (none)
- RV1, RV2: footprint Potentiometer_SMD:Potentiometer_ACP_CA14-VSMD_Vertical -> (none)
Connections:
- net GND renamed 0
